Commit message: Signed-off-by: Or Tslil <ortslil64@gmail.com>

File: gazebo_demo/urdf/ABot.urdf.xacro (robot description, xacro)
@@ -152,14 +152,11 @@
         <friction>
           <ode>
-            <mu>0.01</mu>
-            <mu2>0.01</mu2>
+            <mu>0.000001</mu>
+            <mu2>0.000001</mu2>
           </ode>
         </friction>
       </surface>
   </link>
-  <gazebo reference="back_wheel">
-    <material>Gazebo/White</material>
-  </gazebo>
-  <joint name="base_link_back_wheel" type="continuous">
+   <joint name="base_link_back_wheel" type="fixed">
     <parent link="base_link"/>
     <child link="back_wheel"/>
@@ -167,4 +164,9 @@
     <origin xyz="-0.15 0 0.025"/>
   </joint>
+  <gazebo reference="back_wheel">
+    <material>Gazebo/White</material>
+    <mu1>0.000001</mu1>
+    <mu2>0.000001</mu2>
+  </gazebo>
 <link name="camera_link">
     <collision>
@@ -214,5 +216,5 @@
   </link>
 <joint name="camera_joint" type="fixed">
-    <axis xyz="0 1 0" />
+    <axis xyz="0 0 0" />
     <origin xyz="0.2 0 0.25" rpy="0 0 0"/>
     <parent link="base_link"/>
@@ -244,5 +246,5 @@
       <plugin name="camera_controller" filename="libgazebo_ros_camera.so">
         <alwaysOn>true</alwaysOn>
-        <updateRate>0.0</updateRate>
+        <updateRate>30.0</updateRate>
         <cameraName>/camera</cameraName>
         <imageTopicName>image_raw</imageTopicName>

Commit message: Added a camera above.

File: gazebo_demo/urdf/ABot.urdf.xacro (robot description, xacro)
@@ -189,4 +189,24 @@
     </inertial>
   </link>
+<link name="camera_link_2">
+    <collision>
+      <origin xyz="0 0 0" rpy="0 0 0"/>
+      <geometry>
+    <box size="0.01 0.01 0.01"/>
+      </geometry>
+    </collision>
+    <visual>
+      <origin xyz="0 0 0" rpy="0 0 0"/>
+      <geometry>
+    <box size="0.01 0.01 0.01"/>
+      </geometry>
+      <material name="red"/>
+    </visual>
+    <inertial>
+      <mass value="1e-5" />
+      <origin xyz="0 0 0" rpy="0 0 0"/>
+      <inertia ixx="1e-6" ixy="0" ixz="0" iyy="1e-6" iyz="0" izz="1e-6" />
+    </inertial>
+  </link>
 <joint name="hokuyo_joint" type="fixed">
     <axis xyz="0 1 0" />
@@ -220,4 +240,10 @@
     <parent link="base_link"/>
     <child link="camera_link"/>
+  </joint>
+<joint name="camera_joint_2" type="fixed">
+    <axis xyz="0 0 0" />
+    <origin xyz="0 0 3.3" rpy="0 1.25 0"/>
+    <parent link="base_link"/>
+    <child link="camera_link_2"/>
   </joint>
 <gazebo reference="camera_link">
@@ -251,4 +277,43 @@
         <cameraInfoTopicName>camera_info</cameraInfoTopicName>
         <frameName>camera_link</frameName>
+        <hackBaseline>0.07</hackBaseline>
+        <distortionK1>0.0</distortionK1>
+        <distortionK2>0.0</distortionK2>
+        <distortionK3>0.0</distortionK3>
+        <distortionT1>0.0</distortionT1>
+        <distortionT2>0.0</distortionT2>
+      </plugin>
+    </sensor>
+  </gazebo>
+<gazebo reference="camera_link_2">
+    <sensor type="camera" name="camera_top">
+      <update_rate>30.0</update_rate>
+      <camera name="head_2">
+        <horizontal_fov>1.3962634</horizontal_fov>
+        <image>
+          <width>640</width>
+          <height>480</height>
+          <format>R8G8B8</format>
+        </image>
+        <clip>
+          <near>0.02</near>
+          <far>300</far>
+        </clip>
+        <noise>
+          <type>gaussian</type>
+          <!-- Noise is sampled independently per pixel on each frame.
+               That pixel's noise value is added to each of its color
+               channels, which at that point lie in the range [0,1]. -->
+          <mean>0.0</mean>
+          <stddev>0.007</stddev>
+        </noise>
+      </camera>
+      <plugin name="camera_controller" filename="libgazebo_ros_camera.so">
+        <alwaysOn>true</alwaysOn>
+        <updateRate>30.0</updateRate>
+        <cameraName>/camera_up</cameraName>
+        <imageTopicName>image_raw_up</imageTopicName>
+        <cameraInfoTopicName>camera_info_up</cameraInfoTopicName>
+        <frameName>camera_link_2</frameName>
         <hackBaseline>0.07</hackBaseline>
         <distortionK1>0.0</distortionK1>
@@ -314,3 +379,4 @@
   <xacro:property name="hokuyo_link" value="0.05" />
   <xacro:property name="camera_link" value="0.05" />
+  <xacro:property name="camera_link_2" value="0.05" />
 </robot>

Commit message: Final updates.

File: gazebo_demo/urdf/ABot.urdf.xacro (robot description, xacro)
@@ -27,4 +27,5 @@
   </collision>
   </link>
+<!--
    <link name="box">
   <inertial>
@@ -46,4 +47,7 @@
   </collision>
   </link>
+  <gazebo reference="box">
+    <material>Gazebo/Black</material>
+  </gazebo>
   <joint name="base_link_box" type="fixed">
     <parent link="base_link"/>
@@ -52,6 +56,7 @@
     <origin xyz="-0.05 0 0.225"/>
   </joint>
+-->
   <gazebo reference="base_link">
-    <material>Gazebo/Blue</material>
+    <material>Gazebo/DarkGrey</material>
   </gazebo>
   <link name="right_wheel">
@@ -165,5 +170,5 @@
   </joint>
   <gazebo reference="back_wheel">
-    <material>Gazebo/White</material>
+    <material>Gazebo/Black</material>
     <mu1>0.000001</mu1>
     <mu2>0.000001</mu2>
@@ -189,4 +194,9 @@
     </inertial>
   </link>
+<gazebo reference="camera_link">
+    <material>Gazebo/Black</material>
+    <mu1>0.000001</mu1>
+    <mu2>0.000001</mu2>
+  </gazebo>
 <link name="camera_link_2">
     <collision>
@@ -237,5 +247,5 @@
 <joint name="camera_joint" type="fixed">
     <axis xyz="0 0 0" />
-    <origin xyz="0.2 0 0.25" rpy="0 0 0"/>
+    <origin xyz="0.2 0 0.175" rpy="0 0 0"/>
     <parent link="base_link"/>
     <child link="camera_link"/>
@@ -345,5 +355,5 @@
     <sensor type="gpu_ray" name="head_hokuyo_sensor">
       <pose>0 0 0 0 0 0</pose>
-      <visualize>true</visualize>
+      <visualize>false</visualize>
       <update_rate>10</update_rate>
       <ray>
